File: case/plate/lk7d-plate.kicad_pcb (KiCad board)
At the start: 2 copper layers, 57.1 x 38.1 mm, 6 parts

Commit message: Fix plate export (#7)
Parts:
- CUT3, CUT4, CUT5, CUT6, CUT7, CUT8: moved to B.Cu
