File: pcb/lk7d-pcb.kicad_pcb (KiCad board)
At the start: 2 copper layers, 57.2 x 57.2 mm, 35 parts, among them J1 PINHD_1x4_Male, J2 PINHD_1x4_Male, M1 JLCPCB_2DBarcode_5x5mm, SW1 RotaryEncoder_Switch_MP, SW2 RotaryEncoder_Switch_MP, SW3 SW_Push, SW4 SW_Push, SW5 SW_Push, SW6 SW_Push, SW7 SW_Push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

Commit message: Update LKBD libraries
Parts:
- SW1, SW2: footprint LKBD_KeySwitch:EC11_THT_sqSilk -> LKBD_KeySwitch:ROT_EC11_THT_sqSilk
- U1: footprint LKBD_MCU:MCU_XIAO-RP2040 -> LKBD_MCU:MCU_XIAO_RP2040
